Commit message: fixed position of reference point on table

File: urdf/linearaxis.macro.xacro (robot description, xacro)
@@ -51,5 +51,5 @@
             <child link="${prefix}reference"/>
             <limit effort="1000" velocity="1.0" lower="${axis_bearing_length + axis_table_length/2.}" upper="${axis_length - axis_bearing_length - axis_table_length/2. - axis_gearbox_length}"/>
-            <origin rpy ="0 0 0" xyz="0 ${-axis_width/2.} ${axis_height/2.}"/>
+            <origin rpy ="0 0 0" xyz="0 ${-axis_width/2. - 0.01} ${axis_height/2.-0.016}"/>
         </joint>
     </xacro:macro>

File: urdf/linearaxis.xacro (robot description, xacro)
@@ -7,5 +7,5 @@
   <xacro:include filename="$(find linearaxis_description)/urdf/linearaxis.macro.xacro" ns="la"/>
   <!--Axis Position-->
-  <xacro:la.axis prefix="linear" parent="base_link" size="long">
+  <xacro:la.axis prefix="robot_" parent="base_link" size="long">
     <origin xyz="0 0 0" rpy="0 0 0"/>
   </xacro:la.axis>

Commit message: changed macro name from axis to my_axis because of namespace issues

File: urdf/linearaxis.macro.xacro (robot description, xacro)
@@ -2,5 +2,5 @@
 <robot name="axis"
     xmlns:xacro="http://www.ros.org/wiki/xacro">
-    <xacro:macro name="axis" params="prefix parent size *origin">
+    <xacro:macro name="my_axis" params="prefix parent size *origin">
         <!-- AXIS Details -->
         <xacro:property name="axis_width" value="0.186"/>
@@ -31,6 +31,6 @@
             </collision>
         </link>
-        <!-- Reference -->
-        <link name="${prefix}reference">
+        <!-- Table Reference -->
+        <link name="${prefix}table_reference">
         <visual>
                 <geometry>
@@ -44,10 +44,9 @@
             <parent link="${parent}"/>
             <child link="${prefix}axis"/>
-            <xacro:insert_block name="origin"/>
         </joint>
-        <!-- Axis to Reference -->
-        <joint name="${prefix}axis_to_reference" type="prismatic">
+        <!-- Axis to Table Reference -->
+        <joint name="${prefix}axis_to_table_reference" type="prismatic">
             <parent link="${prefix}axis"/>
-            <child link="${prefix}reference"/>
+            <child link="${prefix}table_reference"/>
             <limit effort="1000" velocity="1.0" lower="${axis_bearing_length + axis_table_length/2.}" upper="${axis_length - axis_bearing_length - axis_table_length/2. - axis_gearbox_length}"/>
             <origin rpy ="0 0 0" xyz="0 ${-axis_width/2. - 0.01} ${axis_height/2.-0.016}"/>

Commit message: added long axis params

File: urdf/linearaxis.macro.xacro (robot description, xacro)
@@ -6,14 +6,20 @@
         <xacro:property name="axis_width" value="0.186"/>
         <xacro:property name="axis_height" value="0.3748"/>
-        <xacro:property name="axis_long_length" value="2.299"/>
+        <xacro:property name="axis_long_length" value="2.6"/>
         <xacro:property name="axis_short_length" value="2.299"/>
-        <xacro:property name="axis_table_length" value="0.28013"/>
-        <xacro:property name="axis_bearing_length" value="0.039"/>
-        <xacro:property name="axis_gearbox_length" value="0.082"/>
+        <xacro:property name="axis_table_length" value="0.2883"/>
+        <xacro:property name="axis_short_bearing_length" value="0.039"/>
+        <xacro:property name="axis_long_bearing_length" value="0.14"/>
+        <xacro:property name="axis_short_gearbox_length" value="0.082"/>
+        <xacro:property name="axis_long_gearbox_length" value="0.0"/>
         <xacro:if value="${size == 'short'}">
             <xacro:property name="axis_length" value="${axis_short_length}"/>
+            <xacro:property name="axis_bearing_length" value="${axis_short_bearing_length}"/>
+            <xacro:property name="axis_gearbox_length" value="${axis_short_gearbox_length}"/>
         </xacro:if>
         <xacro:unless value="${size == 'short'}">
             <xacro:property name="axis_length" value="${axis_long_length}"/>
+            <xacro:property name="axis_bearing_length" value="${axis_long_bearing_length}"/>
+            <xacro:property name="axis_gearbox_length" value="${axis_long_gearbox_length}"/>
         </xacro:unless>
         <!-- AXIS -->

Commit message: first

File: urdf/linearaxis.macro.xacro (robot description, xacro)
@@ -8,4 +8,6 @@
         <xacro:property name="axis_long_length" value="2.6"/>
         <xacro:property name="axis_short_length" value="2.299"/>
+        <xacro:property name="axis_mass" value="1000"/>
+        <xacro:property name="table_reference_mass" value="10"/>
         <xacro:property name="axis_table_length" value="0.2883"/>
         <xacro:property name="axis_short_bearing_length" value="0.039"/>
@@ -23,4 +25,12 @@
             <xacro:property name="axis_gearbox_length" value="${axis_long_gearbox_length}"/>
         </xacro:unless>
+        <xacro:macro name="box_inertial" params="length width height mass">
+            <inertial>
+            <mass value="${mass}" />
+            <inertia ixx="${0.0833333 * mass * (width * width + height * height)}" ixy="0.0" ixz="0.0"
+            iyy="${0.0833333 * mass * (length * length + height * height)}" iyz="0.0"
+            izz="${0.083 * length * length + width * width}" />
+            </inertial>
+        </xacro:macro>
         <!-- AXIS -->
         <link name="${prefix}axis">
@@ -36,5 +46,9 @@
                 </geometry>
             </collision>
+            <box_inertial length="${axis_length}" width="${axis_width}" height="${axis_height}" mass="${axis_mass}"/>
         </link>
+        <gazebo reference="${prefix}axis">
+            <material>Gazebo/Gray</material>
+        </gazebo>
         <!-- Table Reference -->
         <link name="${prefix}table_reference">
@@ -44,5 +58,15 @@
                 </geometry>
         </visual>
+        <collision>
+                <origin xyz="0 0 0" rpy="0 0 0"/>
+                <geometry>
+                    <box size="0.01 0.01 0.01"/>
+                </geometry>
+        </collision>
+        <xacro:box_inertial length="0.1" width="0.1" height="0.1" mass="${table_reference_mass}"/>
         </link>
+        <gazebo reference="${prefix}table_reference">
+            <material>Gazebo/Gray</material>
+        </gazebo>
         <!-- Parent to Axis -->
         <joint name="${parent}to_axis" type="fixed">
